Commit message: modified:   RSEND_Term_2_Project_2_Template__Copy_.pdf 	modified:   udacity_bot/urdf/seans_bot .xacro 	modified:   udacity_bot/urdf/seans_bot.xacro 	udacity_bot/launch/visualize_robot.launch

File: udacity_bot/urdf/seans_bot .xacro (robot description, xacro)
@@ -1,3 +1,4 @@
 <?xml version='1.0'?>
+<!--NOT THIS ONE-->
 <robot name="udacity_bot" xmlns:xacro="http://www.ros.org/wiki/xacro">
   <xacro:include filename="$(find udacity_bot)/urdf/seans_bot.gazebo"/>
@@ -23,5 +24,5 @@
       <origin xyz="0 0 0" rpy=" 0 0 0"/>
       <geometry>
-        <cylinder radius="0.2" length="0.1"/>
+        <cylinder radius="0.2" length="0.6"/>
       </geometry>
     </collision>
@@ -29,5 +30,5 @@
       <origin xyz="0 0 0" rpy=" 0 0 0"/>
       <geometry>
-        <cylinder radius="0.2" length="0.1"/>
+        <cylinder radius="0.2" length="0.6"/>
       </geometry>
       <material name="black">
@@ -190,5 +191,5 @@
     <child link="left_wheel"/>
     <parent link="chassis"/>
-    <axis xyz="0 1 0" rpy="0 0 0"/>
+    <axis xyz="0 0.1 0" rpy="0 0 0"/>
     <limit effort="10000" velocity="1000"/>
     <joint_properties damping="1.0" friction="1.0"/>
@@ -198,5 +199,5 @@
     <child link="right_wheel"/>
     <parent link="chassis"/>
-    <axis xyz="0 1 0" rpy="0 0 0"/>
+    <axis xyz="0 0.1 0" rpy="0 0 0"/>
     <limit effort="10000" velocity="1000"/>
     <joint_properties damping="1.0" friction="1.0"/>

File: udacity_bot/urdf/seans_bot.xacro (robot description, xacro)
@@ -23,5 +23,5 @@
       <origin xyz="0 0 0" rpy=" 0 0 0"/>
       <geometry>
-        <cylinder radius="0.2" length="0.1"/>
+        <cylinder radius="0.2" length="0.6"/>
       </geometry>
     </collision>
@@ -29,5 +29,5 @@
       <origin xyz="0 0 0" rpy=" 0 0 0"/>
       <geometry>
-        <cylinder radius="0.2" length="0.1"/>
+        <cylinder radius="0.2" length="0.6"/>
       </geometry>
       <material name="black">
@@ -36,5 +36,5 @@
     </visual>
     <collision name='back_caster_collision'>
-      <origin xyz="-0.15 0 -0.05" rpy=" 0 0 0"/>
+      <origin xyz="-0.15 0 -0.30" rpy=" 0 0 0"/>
       <geometry>
         <sphere radius="0.0499"/>
@@ -52,5 +52,5 @@
     </collision>
     <visual name='back_caster_visual'>
-      <origin xyz="-0.15 0 -0.05" rpy=" 0 0 0"/>
+      <origin xyz="-0.15 0 -0.30" rpy=" 0 0 0"/>
       <geometry>
         <sphere radius="0.0499"/>
@@ -58,5 +58,5 @@
     </visual>
     <collision name='front_caster_collision'>
-      <origin xyz="0.15 0 -0.05" rpy=" 0 0 0"/>
+      <origin xyz="0.15 0 -0.30" rpy=" 0 0 0"/>
       <geometry>
         <sphere radius="0.0499"/>
@@ -74,5 +74,5 @@
     </collision>
     <visual name='front_caster_visual'>
-      <origin xyz="0.15 0 -0.05" rpy=" 0 0 0"/>
+      <origin xyz="0.15 0 -0.30" rpy=" 0 0 0"/>
       <geometry>
         <sphere radius="0.0499"/>
@@ -93,5 +93,5 @@
     <visual>
       <geometry>
-        <cylinder length="0.05" radius="0.1"/>
+        <cylinder length="0.04" radius="0.0499"/>
       </geometry>
       <origin xyz="0 0 0" rpy="0 1.5707 1.5707"/>
@@ -102,5 +102,5 @@
     <collision>
       <geometry>
-        <cylinder length="0.05" radius="0.1"/>
+        <cylinder length="0.04" radius="0.0499"/>
       </geometry>
       <origin xyz="0 0 0" rpy="0 1.5707 1.5707"/>
@@ -120,5 +120,5 @@
     <visual>
       <geometry>
-        <cylinder length="0.05" radius="0.1"/>
+        <cylinder length="0.04" radius="0.0499"/>
       </geometry>
       <origin xyz="0 0 0" rpy="0 1.5707 1.5707"/>
@@ -129,5 +129,5 @@
     <collision>
       <geometry>
-        <cylinder length="0.05" radius="0.1"/>
+        <cylinder length="0.04" radius="0.0499"/>
       </geometry>
       <origin xyz="0 0 0" rpy="0 1.5707 1.5707"/>
@@ -187,5 +187,5 @@
   <!-- Joints -->
   <joint type="continuous" name="left_wheel_hinge">
-    <origin xyz="0 0.25 0" rpy="0 0 0"/>
+    <origin xyz="0 0.25 -0.30" rpy="0 0 0"/>
     <child link="left_wheel"/>
     <parent link="chassis"/>
@@ -195,5 +195,5 @@
   </joint>
   <joint type="continuous" name="right_wheel_hinge">
-    <origin xyz="0 -0.25 0" rpy="0 0 0"/>
+    <origin xyz="0 -0.25 -0.30" rpy="0 0 0"/>
     <child link="right_wheel"/>
     <parent link="chassis"/>
@@ -208,5 +208,5 @@
   </joint>
   <joint type="fixed" name="hokuyo_joint">
-    <origin xyz="0.0 0 0.1" rpy="0 0 0"/>
+    <origin xyz="0.0 0 0.4" rpy="0 0 0"/>
     <child link="hokuyo"/>
     <parent link="chassis"/>
